File: Clacktronics BYOM Attenuverter/BYOM_Attenuverter_main/BYOM_Attenuverter_main.kicad_pcb (KiCad board)
At the start: 2 copper layers, 29.5 x 100 mm, 20 parts, among them J2 Attenuvert 1, J3 Input 1, J4 Attenuvert 2, J5 Eurorack socket, J6 Input 2, U1 TL074

Commit message: Modifications, added readme
Other:
- board text removed: "CLACKTRONICS"
