File: Clacktronics BYOM Envelope/BYOM_Envelope_main/BYOM_Envelope_main.kicad_pcb (KiCad board)
At the start: 2 copper layers, 29.5 x 100 mm, 24 parts, among them J1 GATE_IN, J2 AR_ENVELOPE_OUT, J3 IDC 02x05 Header, U1 TL074

Commit message: Modifications, added readme
Other:
- board text removed: "CLACKTRONICS"
