File: Clacktronics BYOM Envelope/BYOM_Envelope_main/BYOM_Envelope_main.kicad_sch (KiCad schematic)
At the start: 24 parts, among them J1 GATE_IN, J2 AR_ENVELOPE_OUT, J3 IDC 02x05 Header, U1 TL072

Commit message: Error in envelope schamtic, shows TL072 instead of TL074
Parts:
- U1: value TL072 -> TL074
Changed lines of the file:
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@@
 			)
 		)
-		(property "Value" "TL072"
+		(property "Value" "TL074"
 			(at 158.75 71.5701 0)
 			(effects
@@
 			)
 		)
-		(property "Value" "TL072"
+		(property "Value" "TL074"
 			(at 87.63 67.7601 0)
 			(effects
@@
 			)
 		)
-		(property "Value" "TL072"
+		(property "Value" "TL074"
 			(at 160.02 46.1701 0)
 			(effects
@@
 			)
 		)
-		(property "Value" "TL072"
+		(property "Value" "TL074"
 			(at 88.9 30.48 0)
 			(effects
@@
 			)
 		)
-		(property "Value" "TL072"
+		(property "Value" "TL074"
 			(at 53.34 56.6999 0)
 			(effects
