File: Clacktronics BYOM LFO/BYOM_LFO_main/BYOM_LFO_main.kicad_pcb (KiCad board)
At the start: 2 copper layers, 29.5 x 100 mm, 28 parts, among them J1 SQUARE OUT, J2 SLOPE OUT, J3 Conn_02x05_Odd_Even, U1 TL074

Commit message: Modifications, added readme
Other:
- board text removed: "CLACKTRONICS"
