File: Clacktronics BYOM PSU/BYOM_PSU_main/BYOM_PSU_main.kicad_pcb (KiCad board)
At the start: 2 copper layers, 29.5 x 100 mm, 33 parts, among them J1 +12V, J2 12V Input Screw terminal, J3 -12V, J4 12V input, J5 EURORACK_16_PIN, J6 EURORACK_16_PIN, U1 MC34063AD

Commit message: Modifications, added readme
Other:
- board text removed: "CLACKTRONICS"
