File: Clacktronics BYOM PSU/BYOM_PSU_panel/BYOM_PSU_panel.kicad_pcb (KiCad board)
At the start: 2 copper layers, 30 x 128.5 mm, 8 parts

Commit message: Modifications, added readme
Other:
- board text removed: "CLACKTRONICS"
