File: Clacktronics BYOM Passive mult/BYOM_Passive_mult_main/BYOM_Passive_mult_main.kicad_pcb (KiCad board)
At the start: 2 copper layers, 18.5 x 93 mm, 7 parts, among them J1 AudioJack2_SwitchT, J2 AudioJack2_SwitchT, J3 AudioJack2_SwitchT, J4 AudioJack2_SwitchT, J5 AudioJack2_SwitchT, J6 AudioJack2_SwitchT, J7 AudioJack2_SwitchT

Commit message: Modifications, added readme
Other:
- board text removed: "CLACKTRONICS"
