File: Clacktronics BYOM VCA/BYOM_VCA_main/BYOM_VCA_main.kicad_pcb (KiCad board)
At the start: 2 copper layers, 29.5 x 100 mm, 37 parts, among them J1 AUDIO IN 2, J2 AUDIO_OUT_2, J3 AUDIO IN 1, J4 AUDIO_OUT_1, J5 CV 2, J6 CV 1, J7 Eurorack socket, Q1 2N3906, Q2 2N3906, U1 LM13700

Commit message: Modifications, added readme
Other:
- board text removed: "CLACKTRONICS"
