File: Clacktronics BYOM VCF/BYOM_VCF_main/BYOM_VCF_main.kicad_pcb (KiCad board)
At the start: 2 copper layers, 29.5 x 100 mm, 38 parts, among them J1 AUDIO IN 2, J2 LP OUT, J3 BP OUT, J4 AUDIO IN 1, J5 Eurorack socket, J6 CUTOFF CV, Q1 2N3906, U1 LM13700

Commit message: Modifications, added readme
Other:
- board text removed: "CLACKTRONICS"
