File: Clacktronics BYOM VCO/BYOM_VCO_main/BYOM_VCO_main.kicad_pcb (KiCad board)
At the start: 2 copper layers, 29.5 x 100 mm, 37 parts, among them J1 V/OCT, J2 SAW OUT, J3 IDC 02x05 Header, J4 SYNC_OUT, J5 SYNC_IN, Q1 2N7000, Q2 2N3904, Q3 2N3904, U1 TL074, U2 L78L05_TO92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

Commit message: Modifications, added readme
Other:
- board text removed: "CLACKTRONICS"
