File: Clacktronics BYOM VCO/BYOM_VCO_panel/BYOM_VCO_panel.kicad_pcb (KiCad board)
At the start: 2 copper layers, 30 x 128.5 mm, 2 parts

Commit message: Modifications, added readme
Other:
- board text removed: "CLACKTRONICS"
